File: elec/main_board/compute_module.kicad_sch (KiCad schematic)
At the start: 19 parts, among them J2 Conn_01x22_Female, J3 PinHeader, SW1 TS-1088-AR02016, SW2 TS-1088-AR02016, SW3 TS-1088-AR02016, SW4 TS-1088-AR02016, U1 74LVC1G07SE-7, U18 SL2.1A, Y2 X322512MSB4SI

Commit message: 配線作業中
Signed-off-by: Kazuki Iida <elkel53930@gmail.com>
Parts:
- added R32, R33: RC0201FR-071KL, Resistor_SMD:R_0201_0603Metric, symbol Device:R_Small
Connections:
- net CM3V3 is gone; now on net +3V3CM: J1.2 (VCC)
- net +3V3CM: now also R32.2, R33.2
- net BTN_DOWN: now also Module1.30 (GPIO6); no longer Module1.58 (GPIO2)
- net BTN_LEFT: now also Module1.26 (GPIO19); no longer Module1.54 (GPIO4)
- net BTN_RIGHT: now also Module1.28 (GPIO13); no longer Module1.50 (GPIO17)
- net BTN_UP: now also Module1.24 (GPIO26); no longer Module1.56 (GPIO3)
- net SCL0: now also R32.1
- net SDA0: now also R33.1

Commit message: アートワーク完了
Signed-off-by: Kazuki Iida <elkel53930@gmail.com>
Parts:
- removed C49: RVT1A101M0505, Capacitor_SMD:CP_Elec_5x5.4, symbol Device:C_Polarized_Small
- added C17: CL10A475KO8NNNC, Capacitor_SMD:C_0603_1608Metric, symbol Device:C_Small
- added C48: CL32A107MPVNNNE, Capacitor_SMD:C_1210_3225Metric, symbol Device:C_Small
- added J9: B2B-ZR, Connector_JST:JST_ZH_B2B-ZR_1x02_P1.50mm_Vertical, symbol Connector_Generic:Conn_01x02
- added Q16: IRLML6344, Package_TO_SOT_SMD:SOT-23, symbol Transistor_FET:IRLML2060
- added R37: RC0201FR-0710KL, Resistor_SMD:R_0201_0603Metric, symbol Device:R
Connections:
- net +3V3CM: now also C17.1
- net +5v: now also C48.2
- net GND: now also C17.2, C48.1, Q16.2 (S), R37.1
- net LIGHT: now reaches Module1.25 (GPIO21)
- net LIGHT: now also Q16.1 (G), R37.2
- new net: J9.2 (Pin_2), Q16.3 (D)
- new net +BATT: J9.1 (Pin_1)
- no-connect marks 96 -> 111
