File: elec/main_board/main_board.kicad_sch (KiCad schematic)
At the start: 2 parts

Commit message: アートワーク完了
Signed-off-by: Kazuki Iida <elkel53930@gmail.com>
Other:
- sheet Compute Module ports: added +BATT; removed none
Changed lines of the file:
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@@
+	)
+	(junction
+		(at 231.14 85.09)
+		(diameter 0)
+		(color 0 0 0 0)
 	)
 	(junction
@@
 	(wire
 		(pts
+			(xy 231.14 85.09) (xy 254 85.09)
+		)
+		(stroke
+			(width 0)
+			(type default)
+		)
+	)
+	(wire
+		(pts
 			(xy 147.32 96.52) (xy 147.32 85.09)
 		)
@@
 	(wire
 		(pts
+			(xy 231.14 85.09) (xy 231.14 96.52)
+		)
+		(stroke
+			(width 0)
+			(type default)
+		)
+	)
+	(wire
+		(pts
 			(xy 149.86 87.63) (xy 195.58 87.63)
 		)
@@
 	(wire
 		(pts
-			(xy 198.12 85.09) (xy 254 85.09)
+			(xy 198.12 85.09) (xy 231.14 85.09)
 		)
 		(stroke
@@
 			)
 		)
+		(pin "+BATT" input
+			(at 231.14 96.52 90)
+			(effects
+				(font
+					(size 1.27 1.27)
+				)
+				(justify right)
+			)
+		)
