File: elec/main_board/micromouse.kicad_sch (KiCad schematic)
At the start: 80 parts, among them J4 Conn_01x02, J5 Conn_01x02, J6 B6B-ZR, J7 EncSide, J8 B6B-ZR, J9 EncSide, Q1 DTC114E, Q10 IRLML6344, Q14 MMBT3904, Q2 DTC114E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

Commit message: アートワーク完了
Signed-off-by: Kazuki Iida <elkel53930@gmail.com>
Parts:
- removed C17: CC0603KRX7R9BB104, Capacitor_SMD:C_0402_1005Metric, symbol Device:C_Small
- removed C18: CL05B104KO5NNNC, Capacitor_SMD:C_0402_1005Metric, symbol Device:C_Small
- removed H1, H2, H3, H4: M2 mounting hole, MountingHole:MountingHole_2.2mm_M2, symbol Mechanical:MountingHole
- removed J7, J9: EncSide, Library:EncoderPad, symbol Connector:Conn_01x06_Male
- removed U8, U9: AS5047D, Package_SO:TSSOP-14_4.4x5mm_P0.65mm, symbol Sensor_Magnetic:AS5047D
Connections:
- no-connect marks 40 -> 26
